Commit message: now with a 2D ray plugin

File: urdf/ecn_auv.xacro (robot description, xacro)
@@ -2,114 +2,143 @@
 <!-- STL-version of the URDF, used with gazebo for dynamic simulation  -->
 <robot name="ecn_auv" xmlns:xacro="http://www.ros.org/wiki/xacro">
-<xacro:property name="PI" value="3.1415926535897931"/>
-<!-- Body properties -->
-<xacro:property name="body_mass" value="25"/>
-<xacro:property name="body_radius" value="0.13"/>
-<xacro:property name="body_length" value="1.5" />
-<xacro:property name="X_cob" value="${body_radius*2}" />
-<!-- thrusters -->
-<xacro:property name="tr1" value=".02" />
-<xacro:property name="tl1" value=".1" />
-<xacro:property name="tr2" value=".05" />
-<xacro:property name="tl2" value=".03" />
-<xacro:property name="eps" value="0.00000001"/>
-<!-- Thruster link -->
-<xacro:macro name="thruster_link" params="name xyz rpy">
-    <joint name="${name}" type="fixed">
-        <parent link="base_link"/>
-        <child link="${name}"/>
-        <origin rpy="${rpy}" xyz="${xyz}"/>
-        <dynamics damping="100.0" friction="100.0"/>
-        <limit effort="30" velocity="1.0" lower="-${eps}" upper="${eps}" />
-    </joint>
-    <link name="${name}">
+    <xacro:property name="PI" value="3.1415926535897931"/>
+    <!-- Body properties -->
+    <xacro:property name="body_mass" value="25"/>
+    <xacro:property name="body_radius" value="0.13"/>
+    <xacro:property name="body_length" value="1.5" />
+    <xacro:property name="X_cog" value="${-0.5*body_radius}" />
+    <!-- thrusters -->
+    <xacro:property name="tr1" value=".02" />
+    <xacro:property name="tl1" value=".1" />
+    <xacro:property name="tr2" value=".05" />
+    <xacro:property name="tl2" value=".03" />
+    <xacro:property name="eps" value="0.00000001"/>
+    <!-- Thruster link -->
+    <xacro:macro name="thruster_link" params="name xyz rpy">
+        <joint name="${name}" type="fixed">
+            <parent link="base_link"/>
+            <child link="${name}"/>
+            <origin rpy="${rpy}" xyz="${xyz}"/>
+            <dynamics damping="10.0"/>
+            <axis xyz="0 1 0"/>
+            <limit effort="30" velocity="5.0" lower="-${PI/2}" upper="${PI/2}" />
+        </joint>
+        <link name="${name}">
+            <buoyancy><compensation>1.0</compensation></buoyancy>
             <visual name="${name}_1">
-            <geometry>
-                <cylinder length="${tl1}" radius="${tr1}"/>
-            </geometry>
-            <material name="black">
-                <color rgba="0 0 0 1"/>
-            </material>
+                <geometry>
+                    <cylinder length="${tl1}" radius="${tr1}"/>
+                </geometry>
+                <material name="black">
+                    <color rgba="0 0 0 1"/>
+                </material>
             </visual>
             <visual name="${name}_2">
-            <origin xyz="0 0 -${(tl1+tl2)/2}"/>
-            <geometry>
-                <cylinder length="${tl2}" radius="${tr2}"/>
-            </geometry>
-            <material name="black">
-                <color rgba="0 0 0 1"/>
-            </material>
+                <origin xyz="0 0 -${(tl1+tl2)/2}"/>
+                <geometry>
+                    <cylinder length="${tl2}" radius="${tr2}"/>
+                </geometry>
+                <material name="black">
+                    <color rgba="0 0 0 1"/>
+                </material>
             </visual>
             <inertial>
-        <mass value="${eps}"/>
-        <inertia
-        ixx="${eps}"
-        ixy="0.0"
-        ixz="0.0"
-        iyy="${eps}"
-        iyz="0.0"
-        izz="${eps}"/>
-        </inertial>
-        </link>
-                <gazebo reference="${name}">
-            <material>Gazebo/Black</material>
+                <mass value=".1"/>
+                <inertia
+                    ixx=".1"
+                    ixy="0.0"
+                    ixz="0.0"
+                    iyy=".1"
+                    iyz="0.0"
+                    izz=".1"/>
+                </inertial>
+            </link>
+            <gazebo reference="${name}">
+                <material>Gazebo/Black</material>
+            </gazebo>
+        </xacro:macro>
+        <!-- Plugin list -->
+        <gazebo>
+            <!-- Gazebo plugin listens to the body-->
+            <plugin name="freefloating_gazebo_control" filename="libfreefloating_gazebo_control.so">
+                <switchService>switch</switchService>
+                <updateRate>100</updateRate>
+                <link>base_link</link>
+                <!-- for each thruster, give the map to XYZ+RPY and the maximum effort -->
+                <thruster>
+                    <map>-1 0 0 0 0 ${body_length/3}</map>
+                    <effort>30</effort>
+                </thruster>
+                <thruster>
+                    <map>-1 0 0 0 0 ${-body_length/3}</map>
+                    <effort>30</effort>
+                </thruster>
+                <thruster>
+                    <map>0 1 0 0 0 0</map>
+                    <effort>30</effort>
+                </thruster>
+                <thruster>
+                    <map>0 0 -1 0 ${-0.3*body_length} 0</map>
+                    <effort>30</effort>
+                </thruster>
+                <thruster>
+                    <map>0 0 -1 0 ${0.3*body_length} 0</map>
+                    <effort>30</effort>
+                </thruster>
+            </plugin>
         </gazebo>
-</xacro:macro>
-<!-- Plugin list -->
-    <gazebo>
-    <!-- Gazebo plugin listens to the body-->
-    <plugin name="freefloating_gazebo_control" filename="libfreefloating_gazebo_control.so">
-        <switchService>switch</switchService>
-        <updateRate>100</updateRate>
-        <link>base_link</link>
-        <!-- for each thruster, give the map to XYZ+RPY and the maximum effort -->
-        <thruster>
-            <map>-1 0 0 0 0 ${-body_radius}</map>
-            <effort>30</effort>
-        </thruster>
-        <thruster>
-            <map>-1 0 0 0 0 ${body_radius}</map>
-            <effort>30</effort>
-        </thruster>
-        <thruster>
-            <map>0 1 0 0 0 0</map>
-            <effort>30</effort>
-        </thruster>
-        <thruster>
-            <map>0 0 -1 0 0 0</map>
-            <effort>30</effort>
-        </thruster>
-        <thruster>
-            <map>0 0 -1 0 ${2*X_cob} 0</map>
-            <effort>30</effort>
-        </thruster>
-    </plugin>
-    </gazebo>
-<link name="base_link">
-    <visual>
-    <origin rpy="0 ${-PI/2} 0"/>
-    <geometry>
-        <cylinder length="${body_length}" radius="${body_radius}"/>
-    </geometry>
-    </visual>
-    <inertial>
-        <origin xyz="0 0 -${X_cob}" rpy="0 ${-PI/2} 0"/>
-        <mass value="${body_mass}"/>
-        <inertia
-        ixx="${body_mass*(body_radius*body_radius/4+body_length*body_length/12)}"
-        ixy="0.0"
-        ixz="0.0"
-        iyy="${body_mass*(body_radius*body_radius/4+body_length*body_length/12)}"
-        iyz="0.0"
-        izz="${body_mass*body_radius*body_radius/2}"/>
-        </inertial>
-<buoyancy>
-    <compensation>1.01</compensation>
-    <origin xyz= "0 0 ${X_cob}"/>
-    <limit radius="${body_radius}"/>
-    <damping xyz="60 100 100" rpy="20 50 50"/>
-</buoyancy>
-</link>
+        <link name="base_link">
+            <visual>
+                <origin rpy="0 ${-PI/2} 0"/>
+                <geometry>
+                    <cylinder length="${body_length}" radius="${body_radius}"/>
+                </geometry>
+            </visual>
+            <inertial>
+                <origin xyz="0 0 ${X_cog}" rpy="0 ${-PI/2} 0"/>
+                <mass value="${body_mass}"/>
+                <inertia
+                    ixx="${body_mass*(body_radius*body_radius/4+body_length*body_length/12)}"
+                    ixy="0.0"
+                    ixz="0.0"
+                    iyy="${body_mass*(body_radius*body_radius/4+body_length*body_length/12)}"
+                    iyz="0.0"
+                    izz="${body_mass*body_radius*body_radius/2}"/>
+                </inertial>
+                <buoyancy>
+                    <compensation>1.01</compensation>
+                    <origin xyz= "0 0 0"/>
+                    <limit radius="${body_radius}"/>
+                    <damping xyz="60 100 100" rpy="20 50 50"/>
+                </buoyancy>
+    </link>
+    <!-- example of laser sensor and plugin, publishing to the "sonar" topic -->
+    <gazebo reference="base_link">
+    <sensor name="sonar" type="ray">
+        <visualize>true</visualize>
+        <pose>${body_length/3} 0 0 0 1.570796 0</pose>
+        <update_rate>10</update_rate>
+        <ray>
+        <scan>
+            <horizontal>
+            <samples>290</samples>
+            <resolution>1</resolution>
+            <min_angle>-0.7</min_angle>
+            <max_angle>0.7</max_angle>
+            </horizontal>
+            </scan>
+        <range>
+            <min>.2</min>
+            <max>50</max>
+            <resolution>0.0005</resolution>
+        </range>
+        </ray>
+        <plugin name="sonar_controller" filename="libgazebo_ros_laser.so">
+        <topicName>sonar</topicName>
+        <frameName>base_link</frameName>
+        </plugin>
+    </sensor>
+</gazebo>
     <xacro:thruster_link name="fwd_left" xyz="${-body_length/3} ${body_radius+tr2} 0" rpy="0 ${PI/2} 0"/>
     <xacro:thruster_link name="fwd_right" xyz="${-body_length/3} -${body_radius+tr2} 0" rpy="0 ${PI/2} 0"/>
-</robot>
+        </robot>
